Commit message: v2

File: assembly_v1_description/urdf/materials.xacro (robot description, xacro)
@@ -22,6 +22,3 @@
   <color rgba="0.7686274509803922 0.7725490196078432 0.7686274509803922 1.0"/>
 </material>
-<material name="acciaio_satinato">
-  <color rgba="0.6274509803921569 0.6274509803921569 0.6274509803921569 1.0"/>
-</material>
 </robot>
